File: kicad/led_controller.kicad_pcb (KiCad board)
At the start: 2 copper layers, 60 x 40 mm, 60 parts, among them J1 PWR_IN, J10 Conn_01x04, J2 ADC1, J3 ADC2, J4 ADC3, J5 I2C, J6 UEXT, J7 SPI, J8 5V, J9 UART, Q1 IRF8721PBF-1, Q2 IRF8721PBF-1, Q3 IRF8721PBF-1, SW1 Rotary_Encoder_Switch, SW2 Rotary_Encoder_Switch, SW3 Rotary_Encoder_Switch, SW4 Rotary_Encoder_Switch, SW5 SW_DIP_x01, U1 AP1117-ADJ, U2 Teensy-LC, U3 INA219

Commit message: final commit before seeed, adds gerbers
Connections:
- J6 pad 1: Net-(J6-Pad1) -> +3V3
Routing:
- net +3V3: track 248.4 -> 259.9 mm
- net /TX: track 27.0 -> 28.0 mm
- net /RX: track 26.4 -> 27.1 mm
- net GND: track 55.4 -> 54.8 mm
Other:
- net class Default: clearance 0.25 -> 0.2
- net class PWR: clearance 0.25 -> 0.2
- rule trace_clearance: 0.25 -> 0.2
- board text added: "12V"
- board text added: "3V3"
- board text added: "4B"
- board text added: "5V"
- board text added: "5V SW"
- board text added: "ADC_1"
- board text added: "ADC_2"
- board text added: "ADC_3"
- board text added: "B"
- board text added: "CS"
- board text added: "ENC_1A"
- board text added: "ENC_1B"
- board text added: "ENC_2A"
- board text added: "ENC_2B"
- board text added: "ENC_3A"
- board text added: "ENC_3B"
- board text added: "ENC_4A"
- board text added: "G"
- board text added: "GND"
- board text added: "LED CONTROLLER 2.0V 180603 FITZ"
- board text added: "MISO"
- board text added: "MOSI"
- board text added: "R"
- board text added: "RX"
- board text added: "SCK"
- board text added: "SCL"
- board text added: "SDA"
- board text added: "SW1"
- board text added: "SW2"
- board text added: "SW3"
- board text added: "SW4"
- board text added: "TX"
