File: kicad/led_controller.sch (KiCad schematic (older format))
At the start: 60 parts, among them J1 ISCP_HEADER, J10 CONN_01X01, J11 12V, J12 RED, J13 GREEN, J14 BLUE, J15 CONN_01X01, J16 CONN_01X01, J17 CONN_01X01, J18 CONN_01X01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

Commit message: added arduino libraries
Parts:
- C1, C2, C3, C4, C5, C6, C7, C8, C9: symbol C_Small -> device:C_Small
- J1: symbol CONN_02X03 -> led_controller-rescue:CONN_02X03-RESCUE-led_controller
- J10, J11, J12, J13, J14, J15, J16, J17, J18, J6, J7, J9: symbol CONN_01X01 -> led_controller-rescue:CONN_01X01-RESCUE-led_controller
- J2, J3, J4: symbol CONN_01X03 -> led_controller-rescue:CONN_01X03-RESCUE-led_controller
- J5: symbol CONN_01X04 -> led_controller-rescue:CONN_01X04-RESCUE-led_controller
- J8: symbol CONN_01X02 -> led_controller-rescue:CONN_01X02-RESCUE-led_controller
- Q1, Q2, Q3: symbol IRF8721PBF-1 -> led_controller-rescue:IRF8721PBF-1-RESCUE-led_controller
- R1, R10, R11, R12, R13, R14, R15, R16, R17, R18, R19, R2, R20, R21, R22, R3, R4, R5, R6, R7, R8, R9: symbol RES -> led_controller-rescue:RES-RESCUE-led_controller
- SW1, SW2, SW3, SW4: symbol Rotary_Encoder_Switch -> device:Rotary_Encoder_Switch
- U1: symbol AP1117-33 -> regul:AP1117-33
- U2: symbol ATMEGA328P-AU -> atmel:ATMEGA328P-AU
- U3: symbol INA219 -> led_controller-rescue:INA219-RESCUE-led_controller
- Y1: symbol Crystal_Small -> device:Crystal_Small
Connections:
- wire segments 225 -> 287

Commit message: switches to kicad and updates schematic and footprints
Parts:
- removed C1: 0.1uF, Capacitors_SMD:C_0805, symbol device:C_Small
- removed C2, C3, C4, C6, C9: 0.1uF, Capacitors_SMD:C_0402, symbol device:C_Small
- removed C5: 10uF, Capacitors_SMD:C_0805, symbol device:C_Small
- removed C7, C8: 22pF, Capacitors_SMD:C_0402, symbol device:C_Small
- removed J1: ISCP_HEADER, Pin_Headers:Pin_Header_Straight_2x03_Pitch2.54mm, symbol led_controller-rescue:CONN_02X03-RESCUE-led_controller
- removed J10, J6, J7, J9: CONN_01X01, Pin_Headers:Pin_Header_Straight_1x01_Pitch2.54mm, symbol led_controller-rescue:CONN_01X01-RESCUE-led_controller
- removed J11: 12V, Pin_Headers:Pin_Header_Straight_1x01_Pitch2.54mm, symbol led_controller-rescue:CONN_01X01-RESCUE-led_controller
- removed J12: RED, Pin_Headers:Pin_Header_Straight_1x01_Pitch2.54mm, symbol led_controller-rescue:CONN_01X01-RESCUE-led_controller
- removed J13: GREEN, Pin_Headers:Pin_Header_Straight_1x01_Pitch2.54mm, symbol led_controller-rescue:CONN_01X01-RESCUE-led_controller
- removed J14: BLUE, Pin_Headers:Pin_Header_Straight_1x01_Pitch2.54mm, symbol led_controller-rescue:CONN_01X01-RESCUE-led_controller
- removed J15, J16, J17, J18: CONN_01X01, Mounting_Holes:MountingHole_2.2mm_M2, symbol led_controller-rescue:CONN_01X01-RESCUE-led_controller
- removed SW1, SW2, SW3, SW4: Rotary_Encoder_Switch, Pin_Headers:Pin_Header_Straight_1x05_Pitch2.54mm, symbol device:Rotary_Encoder_Switch
- removed U1: AP1117-33, TO_SOT_Packages_SMD:SOT-223-3Lead_TabPin2, symbol regul:AP1117-33
- removed U2: ATMEGA328P-AU, Housings_QFP:TQFP-32_7x7mm_Pitch0.8mm, symbol atmel:ATMEGA328P-AU
- removed Y1: 16Mhz, Crystals:Crystal_SMD_HC49-SD, symbol device:Crystal_Small
- added C1, C2: 10uF, Capacitor_SMD:C_0603_1608Metric, symbol Device:C_Small
- added C3: 0.1uF, Capacitor_SMD:C_0402_1005Metric, symbol Device:C_Small
- added J1: PWR_IN, Connector_Phoenix_MC:PhoenixContact_MCV_1,5_2-G-5.08_1x02_P5.08mm_Vertical, symbol Connector_Generic:Conn_01x02
- added J10: Conn_01x04, Connector_Phoenix_MC:PhoenixContact_MCV_1,5_4-G-5.08_1x04_P5.08mm_Vertical, symbol Connector_Generic:Conn_01x04
- added J6: UEXT, Connector_PinHeader_2.54mm:PinHeader_2x05_P2.54mm_Vertical, symbol Connector_Generic:Conn_02x05_Odd_Even
- added J7: SPI, Connector_JST:JST_SH_BM05B-SRSS-TB_1x05-1MP_P1.00mm_Vertical, symbol Connector_Generic:Conn_01x05
- added J9: UART, Connector_JST:JST_SH_SM04B-SRSS-TB_1x04-1MP_P1.00mm_Horizontal, symbol Connector_Generic:Conn_01x04
- added JP1, JP2: Jumper_NC_Small, Jumper:SolderJumper-2_P1.3mm_Bridged_RoundedPad1.0x1.5mm, symbol Device:Jumper_NC_Small
- added MK? (x4): Mounting_Hole, MountingHole:MountingHole_2.2mm_M2, symbol Mechanical:Mounting_Hole
- added R23, R24, R25, R26, R27: 10K, Resistor_SMD:R_0402_1005Metric, symbol led_controller-rescue:RES-RESCUE-led_controller
- added R28, R29, R30: 0R1, Resistor_SMD:R_1206_3216Metric, symbol led_controller-rescue:RES-RESCUE-led_controller
- added SW1, SW2, SW3, SW4: Rotary_Encoder_Switch, Connector_JST:JST_SH_SM05B-SRSS-TB_1x05-1MP_P1.00mm_Horizontal, symbol Device:Rotary_Encoder_Switch
- added SW5: SW_DIP_x01, Connector_PinSocket_2.54mm:PinSocket_1x02_P2.54mm_Vertical, symbol Switch:SW_DIP_x01
- added U1: AP1117-ADJ, Package_TO_SOT_SMD:SOT-223-3_TabPin2, symbol Regulator_Linear:AP1117-ADJ
- added U2: Teensy-LC, teensy:Teensy30_31_32_LC, symbol teensy:Teensy-LC
- J2: value CONN_01X03 -> ADC1
- J3: value CONN_01X03 -> ADC2
- J4: value CONN_01X03 -> ADC3
- J5: value OLED -> I2C; footprint Pin_Headers:Pin_Header_Straight_1x04_Pitch2.54mm -> Connector_JST:JST_SH_SM04B-SRSS-TB_1x04-1MP_P1.00mm_Horizontal
- J8: value CONN_01X02 -> 5V
- R1, R10, R11, R13, R14, R15, R16, R17, R18, R19, R2, R20, R21, R22, R3, R4, R5, R6, R7, R8, R9: footprint Resistors_SMD:R_0402 -> Resistor_SMD:R_0402_1005Metric
- R12: footprint Resistors_SMD:R_1206_HandSoldering -> Resistor_SMD:R_1206_3216Metric
Connections:
- net labels added: +5V, CS0, MISO0, MOSI0, SCK0, SCL, SDA, SW1, SW2, SW3, SW4
- wire segments 287 -> 307
Other:
- note removed: "OLED DISPLAY"
- note removed: "PLACE DECOUPLING CAPS CLOSE TO ATMEGA"

Commit message: finishes placement and power routing
Parts:
- removed SW1, SW2, SW3, SW4: Rotary_Encoder_Switch, Connector_JST:JST_SH_SM05B-SRSS-TB_1x05-1MP_P1.00mm_Horizontal, symbol Device:Rotary_Encoder_Switch
- added SW1, SW2, SW3, SW4: Rotary_Encoder_Switch, Connector_JST:JST_SH_BM05B-SRSS-TB_1x05-1MP_P1.00mm_Vertical, symbol led_controller:Rotary_Encoder_Switch
- J2, J3, J4: footprint Pin_Headers:Pin_Header_Straight_1x03_Pitch2.54mm -> Connector_JST:JST_SH_SM03B-SRSS-TB_1x03-1MP_P1.00mm_Horizontal
- gave numbers to parts that had none: 4
Connections:
- net labels added: 12V_SHUNT, 5V_SW
Changed lines of the file:
@@
 Comment4 ""
 $EndDescr
+Text Label 7200 4300 0    60   ~ 0
+RX
 Text Label 7200 4200 0    60   ~ 0
-RX
-Text Label 7200 4300 0    60   ~ 0
 TX
 $Comp
@@
 F 0 "J4" H 9128 3541 50  0000 L CNN
 F 1 "ADC3" H 9128 3450 50  0001 L CNN
-F 2 "Pin_Headers:Pin_Header_Straight_1x03_Pitch2.54mm" H 9050 3500 50  0001 C CNN
+F 2 "Connector_JST:JST_SH_SM03B-SRSS-TB_1x03-1MP_P1.00mm_Horizontal" H 9050 3500 50  0001 C CNN
 F 3 "" H 9050 3500 50  0001 C CNN
 	1    9050 3500
@@
 F 0 "J3" H 9128 2541 50  0000 L CNN
 F 1 "ADC2" H 9128 2450 50  0001 L CNN
-F 2 "Pin_Headers:Pin_Header_Straight_1x03_Pitch2.54mm" H 9050 2500 50  0001 C CNN
+F 2 "Connector_JST:JST_SH_SM03B-SRSS-TB_1x03-1MP_P1.00mm_Horizontal" H 9050 2500 50  0001 C CNN
 F 3 "" H 9050 2500 50  0001 C CNN
 	1    9050 2500
@@
 F 0 "J2" H 9128 1491 50  0000 L CNN
 F 1 "ADC1" H 9128 1400 50  0001 L CNN
-F 2 "Pin_Headers:Pin_Header_Straight_1x03_Pitch2.54mm" H 9050 1450 50  0001 C CNN
+F 2 "Connector_JST:JST_SH_SM03B-SRSS-TB_1x03-1MP_P1.00mm_Horizontal" H 9050 1450 50  0001 C CNN
 F 3 "" H 9050 1450 50  0001 C CNN
 	1    9050 1450
@@
 F 3 "" H 2950 4000 60  0000 C CNN
 	1    2950 4550
-	1    0    0    -1
-$EndComp
-$Comp
-L Device:Rotary_Encoder_Switch SW3
-U 1 1 5B12BF59
-P 11250 4250
-F 0 "SW3" H 11250 4617 50  0000 C CNN
-F 1 "Rotary_Encoder_Switch" H 11250 4526 50  0000 C CNN
-F 2 "Connector_JST:JST_SH_SM05B-SRSS-TB_1x05-1MP_P1.00mm_Horizontal" H 11100 4410 50  0001 C CNN
-F 3 "~" H 11250 4510 50  0001 C CNN
-	1    11250 4250
-	1    0    0    -1
-$EndComp
-$Comp
-L Device:Rotary_Encoder_Switch SW2
-U 1 1 5B12C19B
-P 11250 2300
-F 0 "SW2" H 11250 2667 50  0000 C CNN
-F 1 "Rotary_Encoder_Switch" H 11250 2576 50  0000 C CNN
-F 2 "Connector_JST:JST_SH_SM05B-SRSS-TB_1x05-1MP_P1.00mm_Horizontal" H 11100 2460 50  0001 C CNN
-F 3 "~" H 11250 2560 50  0001 C CNN
-	1    11250 2300
-	1    0    0    -1
-$EndComp
-$Comp
-L Device:Rotary_Encoder_Switch SW4
-U 1 1 5B12C22F
-P 11250 6150
-F 0 "SW4" H 11250 6517 50  0000 C CNN
-F 1 "Rotary_Encoder_Switch" H 11250 6426 50  0000 C CNN
-F 2 "Connector_JST:JST_SH_SM05B-SRSS-TB_1x05-1MP_P1.00mm_Horizontal" H 11100 6310 50  0001 C CNN
-F 3 "~" H 11250 6410 50  0001 C CNN
-	1    11250 6150
-	1    0    0    -1
-$EndComp
-$Comp
-L Device:Rotary_Encoder_Switch SW1
-U 1 1 5B12C2D1
-P 11200 8150
-F 0 "SW1" H 11200 8517 50  0000 C CNN
-F 1 "Rotary_Encoder_Switch" H 11200 8426 50  0000 C CNN
-F 2 "Connector_JST:JST_SH_SM05B-SRSS-TB_1x05-1MP_P1.00mm_Horizontal" H 11050 8310 50  0001 C CNN
-F 3 "~" H 11200 8410 50  0001 C CNN
-	1    11200 8150
 	1    0    0    -1
 $EndComp
@@
 	4250 1200 4250 1300
 $Comp
-L Mechanical:Mounting_Hole MK?
+L Mechanical:Mounting_Hole MK1
 U 1 1 5BA52F5B
 P 1600 7200
-F 0 "MK?" H 1700 7246 50  0000 L CNN
+F 0 "MK1" H 1700 7246 50  0000 L CNN
 F 1 "Mounting_Hole" H 1700 7155 50  0000 L CNN
 F 2 "MountingHole:MountingHole_2.2mm_M2" H 1600 7200 50  0001 C CNN
@@
 $EndComp
 $Comp
-L Mechanical:Mounting_Hole MK?
+L Mechanical:Mounting_Hole MK3
 U 1 1 5BA53363
 P 2600 7200
-F 0 "MK?" H 2700 7246 50  0000 L CNN
+F 0 "MK3" H 2700 7246 50  0000 L CNN
 F 1 "Mounting_Hole" H 2700 7155 50  0000 L CNN
 F 2 "MountingHole:MountingHole_2.2mm_M2" H 2600 7200 50  0001 C CNN
@@
 $EndComp
 $Comp
-L Mechanical:Mounting_Hole MK?
+L Mechanical:Mounting_Hole MK2
 U 1 1 5BA5341F
 P 1600 7550
-F 0 "MK?" H 1700 7596 50  0000 L CNN
+F 0 "MK2" H 1700 7596 50  0000 L CNN
 F 1 "Mounting_Hole" H 1700 7505 50  0000 L CNN
 F 2 "MountingHole:MountingHole_2.2mm_M2" H 1600 7550 50  0001 C CNN
@@
 $EndComp
 $Comp
-L Mechanical:Mounting_Hole MK?
+L Mechanical:Mounting_Hole MK4
 U 1 1 5BA5350D
 P 2600 7550
-F 0 "MK?" H 2700 7596 50  0000 L CNN
+F 0 "MK4" H 2700 7596 50  0000 L CNN
 F 1 "Mounting_Hole" H 2700 7505 50  0000 L CNN
 F 2 "MountingHole:MountingHole_2.2mm_M2" H 2600 7550 50  0001 C CNN
@@
 	1    0    0    -1
 $EndComp
+$Comp
+L led_controller:Rotary_Encoder_Switch SW4
+U 1 1 5B15CC18
+P 11200 8150
+F 0 "SW4" H 11200 8517 50  0000 C CNN
+F 1 "Rotary_Encoder_Switch" H 11200 8426 50  0000 C CNN
+F 2 "Connector_JST:JST_SH_BM05B-SRSS-TB_1x05-1MP_P1.00mm_Vertical" H 11050 8310 50  0001 C CNN
+F 3 "~" H 11200 8410 50  0001 C CNN
+	1    11200 8150
+	1    0    0    -1
+$EndComp
+$Comp
+L led_controller:Rotary_Encoder_Switch SW3
+U 1 1 5B15D1C9
+P 11250 6150
+F 0 "SW3" H 11250 6517 50  0000 C CNN
+F 1 "Rotary_Encoder_Switch" H 11250 6426 50  0000 C CNN
+F 2 "Connector_JST:JST_SH_BM05B-SRSS-TB_1x05-1MP_P1.00mm_Vertical" H 11100 6310 50  0001 C CNN
+F 3 "~" H 11250 6410 50  0001 C CNN
+	1    11250 6150
+	1    0    0    -1
+$EndComp
+$Comp
+L led_controller:Rotary_Encoder_Switch SW2
+U 1 1 5B15D2BB
+P 11250 4250
+F 0 "SW2" H 11250 4617 50  0000 C CNN
+F 1 "Rotary_Encoder_Switch" H 11250 4526 50  0000 C CNN
+F 2 "Connector_JST:JST_SH_BM05B-SRSS-TB_1x05-1MP_P1.00mm_Vertical" H 11100 4410 50  0001 C CNN
+F 3 "~" H 11250 4510 50  0001 C CNN
+	1    11250 4250
+	1    0    0    -1
+$EndComp
+$Comp
+L led_controller:Rotary_Encoder_Switch SW1
+U 1 1 5B15D4DD
+P 11250 2300
+F 0 "SW1" H 11250 2667 50  0000 C CNN
+F 1 "Rotary_Encoder_Switch" H 11250 2576 50  0000 C CNN
+F 2 "Connector_JST:JST_SH_BM05B-SRSS-TB_1x05-1MP_P1.00mm_Vertical" H 11100 2460 50  0001 C CNN
+F 3 "~" H 11250 2560 50  0001 C CNN
+	1    11250 2300
+	1    0    0    -1
+$EndComp
+Text Label 14150 6500 0    50   ~ 0
+12V_SHUNT
+Text Label 2950 1200 0    50   ~ 0
+5V_SW
 $EndSCHEMATC

Commit message: finishes layout, needs look over and silk
Connections:
- net labels added: OUT_B, OUT_G, OUT_R
- net labels removed: I2C_SCL, I2C_SDA
- wire segments 307 -> 309
Changed lines of the file:
@@
 Text Label 8400 1450 2    60   ~ 0
 ADC_1
-Text Label 4350 5300 0    60   ~ 0
+Text Label 4350 3900 0    60   ~ 0
 ADC_2
 Wire Wire Line
@@
 Wire Wire Line
 	4350 5300 4050 5300
-Text Label 4350 5200 0    60   ~ 0
+Text Label 4350 4000 0    60   ~ 0
 ADC_3
 Wire Wire Line
@@
 Text Label 10200 8250 2    60   ~ 0
 ENC_4B
-Text Label 1800 3900 2    60   ~ 0
+Text Label 1800 4100 2    60   ~ 0
 ENC_1A
 Text Label 1800 4000 2    60   ~ 0
 ENC_1B
-Text Label 1800 4100 2    60   ~ 0
+Text Label 4350 4800 0    60   ~ 0
 ENC_2A
-Text Label 1800 4200 2    60   ~ 0
+Text Label 1800 4400 2    60   ~ 0
 ENC_3A
 Text Label 1800 4300 2    60   ~ 0
 ENC_3B
-Text Label 1800 4400 2    60   ~ 0
+Text Label 4350 5500 0    60   ~ 0
 ENC_4A
-Text Label 1800 4500 2    60   ~ 0
+Text Label 1800 4600 2    60   ~ 0
 ENC_4B
 Wire Wire Line
@@
 Text Label 4350 4900 0    60   ~ 0
 PWM_R
-Text Label 4350 4700 0    60   ~ 0
+Text Label 4350 5200 0    60   ~ 0
 PWM_G
-Text Label 4350 4600 0    60   ~ 0
+Text Label 4350 5300 0    60   ~ 0
 PWM_B
 Wire Wire Line
@@
 Wire Wire Line
 	4050 5500 4350 5500
-Text Label 4350 5500 0    50   ~ 0
+Text Label 1800 5500 2    50   ~ 0
 SCK0
 Text Label 1800 4700 2    50   ~ 0
@@
 	7300 8550 7400 8550
 Text Label 14000 8950 2    60   ~ 0
-I2C_SDA
+SDA
 $Comp
 L Device:Jumper_NC_Small JP1
@@
 $EndComp
 Text Label 14350 9000 3    60   ~ 0
-I2C_SCL
+SCL
 Wire Wire Line
 	14350 9000 14350 8800
@@
 Wire Wire Line
 	4150 4400 4050 4400
-Text Label 1800 4600 2    50   ~ 0
+Text Label 1800 3900 2    50   ~ 0
 SW1
 Wire Wire Line
 	1900 4600 1800 4600
-Text Label 1800 5400 2    50   ~ 0
+Text Label 4350 4600 0    50   ~ 0
 SW2
 Wire Wire Line
 	1800 5400 1900 5400
-Text Label 4350 4800 0    50   ~ 0
+Text Label 1800 4200 2    50   ~ 0
 SW3
 Wire Wire Line
 	4350 4800 4050 4800
-Text Label 4350 4000 0    50   ~ 0
+Text Label 1800 4500 2    50   ~ 0
 SW4
 Wire Wire Line
@@
 Text Label 2950 1200 0    50   ~ 0
 5V_SW
+Text Label 4350 4700 0    60   ~ 0
+ENC_2B
+Wire Wire Line
+	1900 5500 1800 5500
+Wire Wire Line
+	4350 3900 4050 3900
+Text Label 14050 1000 0    50   ~ 0
+OUT_R
+Text Label 14100 2800 0    50   ~ 0
+OUT_G
+Text Label 14150 4300 0    50   ~ 0
+OUT_B
 $EndSCHEMATC

Commit message: final commit before seeed, adds gerbers
Changed lines of the file:
@@
 Text Label 14150 4300 0    50   ~ 0
 OUT_B
+$Comp
+L power:+3V3 #PWR?
+U 1 1 5B1684B7
+P 7000 5100
+F 0 "#PWR?" H 7000 4950 50  0001 C CNN
+F 1 "+3V3" H 7015 5273 50  0000 C CNN
+F 2 "" H 7000 5100 50  0001 C CNN
+F 3 "" H 7000 5100 50  0001 C CNN
+	1    7000 5100
+	1    0    0    -1
+$EndComp
 $EndSCHEMATC
